Commit message: Update Gazebo and controller configurations

File: robotic_arm/urdf/robotic_arm_2.urdf.xacro (robot description, xacro)
@@ -4,5 +4,5 @@
      Commit Version: 1.5.1-0-g916b5db  Build Version: 1.5.7152.31018
      For more information, please see http://wiki.ros.org/sw_urdf_exporter -->
-<robot
+<robot xmlns:xacro="https://wiki.ros.org/xacro.org"
   name="robotic_arm">
   <link name="world" />
@@ -35,19 +35,19 @@
       <geometry>
         <mesh
-          filename="package://robotic_arm/meshes/base_link.STL" />
-      </geometry>
-      <material
-        name="">
-        <color
-          rgba="0.501960784313725 0.501960784313725 0.501960784313725 1" />
-      </material>
-    </visual>
-    <collision>
-      <origin
-        xyz="0 0 0"
-        rpy="0 0 0" />
-      <geometry>
-        <mesh
-          filename="package://robotic_arm/meshes/base_link.STL" />
+          filename="file://$(find robotic_arm)/meshes/base_link.STL" />
+      </geometry>
+      <material
+        name="">
+        <color
+          rgba="0.501960784313725 0.501960784313725 0.501960784313725 1" />
+      </material>
+    </visual>
+    <collision>
+      <origin
+        xyz="0 0 0"
+        rpy="0 0 0" />
+      <geometry>
+        <mesh
+          filename="file://$(find robotic_arm)/meshes/base_link.STL" />
       </geometry>
     </collision>
@@ -76,19 +76,19 @@
       <geometry>
         <mesh
-          filename="package://robotic_arm/meshes/link_1.STL" />
-      </geometry>
-      <material
-        name="">
-        <color
-          rgba="0.501960784313725 0.501960784313725 0.501960784313725 1" />
-      </material>
-    </visual>
-    <collision>
-      <origin
-        xyz="0 0 0"
-        rpy="0 0 0" />
-      <geometry>
-        <mesh
-          filename="package://robotic_arm/meshes/link_1.STL" />
+          filename="file://$(find robotic_arm)/meshes/link_1.STL" />
+      </geometry>
+      <material
+        name="">
+        <color
+          rgba="0.501960784313725 0.501960784313725 0.501960784313725 1" />
+      </material>
+    </visual>
+    <collision>
+      <origin
+        xyz="0 0 0"
+        rpy="0 0 0" />
+      <geometry>
+        <mesh
+          filename="file://$(find robotic_arm)/meshes/link_1.STL" />
       </geometry>
     </collision>
@@ -110,5 +110,5 @@
       upper="6.283"
       effort="300"
-      velocity="3" />
+      velocity="3.14" />
   </joint>
   <link
@@ -135,19 +135,19 @@
       <geometry>
         <mesh
-          filename="package://robotic_arm/meshes/link_2.STL" />
-      </geometry>
-      <material
-        name="">
-        <color
-          rgba="0.501960784313725 0.501960784313725 0.501960784313725 1" />
-      </material>
-    </visual>
-    <collision>
-      <origin
-        xyz="0 0 0"
-        rpy="0 0 0" />
-      <geometry>
-        <mesh
-          filename="package://robotic_arm/meshes/link_2.STL" />
+          filename="file://$(find robotic_arm)/meshes/link_2.STL" />
+      </geometry>
+      <material
+        name="">
+        <color
+          rgba="0.501960784313725 0.501960784313725 0.501960784313725 1" />
+      </material>
+    </visual>
+    <collision>
+      <origin
+        xyz="0 0 0"
+        rpy="0 0 0" />
+      <geometry>
+        <mesh
+          filename="file://$(find robotic_arm)/meshes/link_2.STL" />
       </geometry>
     </collision>
@@ -169,5 +169,5 @@
       upper="1.57"
       effort="300"
-      velocity="3" />
+      velocity="3.14" />
   </joint>
   <link
@@ -194,19 +194,19 @@
       <geometry>
         <mesh
-          filename="package://robotic_arm/meshes/link_3.STL" />
-      </geometry>
-      <material
-        name="">
-        <color
-          rgba="0.501960784313725 0.501960784313725 0.501960784313725 1" />
-      </material>
-    </visual>
-    <collision>
-      <origin
-        xyz="0 0 0"
-        rpy="0 0 0" />
-      <geometry>
-        <mesh
-          filename="package://robotic_arm/meshes/link_3.STL" />
+          filename="file://$(find robotic_arm)/meshes/link_3.STL" />
+      </geometry>
+      <material
+        name="">
+        <color
+          rgba="0.501960784313725 0.501960784313725 0.501960784313725 1" />
+      </material>
+    </visual>
+    <collision>
+      <origin
+        xyz="0 0 0"
+        rpy="0 0 0" />
+      <geometry>
+        <mesh
+          filename="file://$(find robotic_arm)/meshes/link_3.STL" />
       </geometry>
     </collision>
@@ -228,5 +228,5 @@
       upper="4.14"
       effort="300"
-      velocity="3" />
+      velocity="3.14" />
   </joint>
   <link
@@ -253,19 +253,19 @@
       <geometry>
         <mesh
-          filename="package://robotic_arm/meshes/link_4.STL" />
-      </geometry>
-      <material
-        name="">
-        <color
-          rgba="0.501960784313725 0.501960784313725 0.501960784313725 1" />
-      </material>
-    </visual>
-    <collision>
-      <origin
-        xyz="0 0 0"
-        rpy="0 0 0" />
-      <geometry>
-        <mesh
-          filename="package://robotic_arm/meshes/link_4.STL" />
+          filename="file://$(find robotic_arm)/meshes/link_4.STL" />
+      </geometry>
+      <material
+        name="">
+        <color
+          rgba="0.501960784313725 0.501960784313725 0.501960784313725 1" />
+      </material>
+    </visual>
+    <collision>
+      <origin
+        xyz="0 0 0"
+        rpy="0 0 0" />
+      <geometry>
+        <mesh
+          filename="file://$(find robotic_arm)/meshes/link_4.STL" />
       </geometry>
     </collision>
@@ -287,5 +287,5 @@
       upper="2.14"
       effort="300"
-      velocity="3" />
+      velocity="3.14" />
   </joint>
   <link
@@ -312,19 +312,19 @@
       <geometry>
         <mesh
-          filename="package://robotic_arm/meshes/link_5.STL" />
-      </geometry>
-      <material
-        name="">
-        <color
-          rgba="0.501960784313725 0.501960784313725 0.501960784313725 1" />
-      </material>
-    </visual>
-    <collision>
-      <origin
-        xyz="0 0 0"
-        rpy="0 0 0" />
-      <geometry>
-        <mesh
-          filename="package://robotic_arm/meshes/link_5.STL" />
+          filename="file://$(find robotic_arm)/meshes/link_5.STL" />
+      </geometry>
+      <material
+        name="">
+        <color
+          rgba="0.501960784313725 0.501960784313725 0.501960784313725 1" />
+      </material>
+    </visual>
+    <collision>
+      <origin
+        xyz="0 0 0"
+        rpy="0 0 0" />
+      <geometry>
+        <mesh
+          filename="file://$(find robotic_arm)/meshes/link_5.STL" />
       </geometry>
     </collision>
@@ -346,5 +346,5 @@
       upper="6.283"
       effort="300"
-      velocity="3" />
+      velocity="3.14" />
   </joint>
   <link
@@ -371,19 +371,19 @@
       <geometry>
         <mesh
-          filename="package://robotic_arm/meshes/eef_link_r.STL" />
-      </geometry>
-      <material
-        name="">
-        <color
-          rgba="0.501960784313725 0.501960784313725 0.501960784313725 1" />
-      </material>
-    </visual>
-    <collision>
-      <origin
-        xyz="0 0 0"
-        rpy="0 0 0" />
-      <geometry>
-        <mesh
-          filename="package://robotic_arm/meshes/eef_link_r.STL" />
+          filename="file://$(find robotic_arm)/meshes/eef_link_r.STL" />
+      </geometry>
+      <material
+        name="">
+        <color
+          rgba="0.501960784313725 0.501960784313725 0.501960784313725 1" />
+      </material>
+    </visual>
+    <collision>
+      <origin
+        xyz="0 0 0"
+        rpy="0 0 0" />
+      <geometry>
+        <mesh
+          filename="file://$(find robotic_arm)/meshes/eef_link_r.STL" />
       </geometry>
     </collision>
@@ -405,5 +405,5 @@
       upper="0.3"
       effort="300"
-      velocity="3" />
+      velocity="3.14" />
   </joint>
   <link
@@ -430,19 +430,19 @@
       <geometry>
         <mesh
-          filename="package://robotic_arm/meshes/eef_link_l.STL" />
-      </geometry>
-      <material
-        name="">
-        <color
-          rgba="0.501960784313725 0.501960784313725 0.501960784313725 1" />
-      </material>
-    </visual>
-    <collision>
-      <origin
-        xyz="0 0 0"
-        rpy="0 0 0" />
-      <geometry>
-        <mesh
-          filename="package://robotic_arm/meshes/eef_link_l.STL" />
+          filename="file://$(find robotic_arm)/meshes/eef_link_l.STL" />
+      </geometry>
+      <material
+        name="">
+        <color
+          rgba="0.501960784313725 0.501960784313725 0.501960784313725 1" />
+      </material>
+    </visual>
+    <collision>
+      <origin
+        xyz="0 0 0"
+        rpy="0 0 0" />
+      <geometry>
+        <mesh
+          filename="file://$(find robotic_arm)/meshes/eef_link_l.STL" />
       </geometry>
     </collision>
@@ -464,5 +464,5 @@
       upper="0.3"
       effort="300"
-      velocity="3" />
+      velocity="3.14" />
   </joint>
   <transmission name="link_1_trans">
@@ -526,17 +526,10 @@
     </actuator>
   </transmission>
-  <ros2_control name="ros2_control" type="system">
+  <ros2_control name="GazeboSimSystem" type="system">
     <hardware>
-      <plugin>gazebo_ros2_control/GazeboSystem</plugin>
+      <plugin>mock_components/GenericSystem</plugin>
     </hardware>
     <joint name="joint_1">
-      <command_interface name="position">
-        <param name="min">0</param>
-        <param name="max">6.283</param>
-      </command_interface>
-      <command_interface name="velocity">
-        <param name="min">-3.15</param>
-        <param name="max">3.15</param>
-      </command_interface>
+      <command_interface name="position" />
       <state_interface name="position">
         <param name="initial_value">0.0</param>
@@ -545,12 +538,5 @@
     </joint>
     <joint name="joint_2">
-      <command_interface name="position">
-        <param name="min">-1.57</param>
-        <param name="max">1.57</param>
-      </command_interface>
-      <command_interface name="velocity">
-        <param name="min">-3.15</param>
-        <param name="max">3.15</param>
-      </command_interface>
+      <command_interface name="position" />
       <state_interface name="position">
         <param name="initial_value">0.0</param>
@@ -559,12 +545,5 @@
     </joint>
     <joint name="joint_3">
-      <command_interface name="position">
-        <param name="min">-1.0</param>
-        <param name="max">4.14</param>
-      </command_interface>
-      <command_interface name="velocity">
-        <param name="min">-3.15</param>
-        <param name="max">3.15</param>
-      </command_interface>
+      <command_interface name="position" />
       <state_interface name="position">
         <param name="initial_value">0.0</param>
@@ -573,12 +552,5 @@
     </joint>
     <joint name="joint_4">
-      <command_interface name="position">
-        <param name="min">-2.14</param>
-        <param name="max">2.14</param>
-      </command_interface>
-      <command_interface name="velocity">
-        <param name="min">-3.15</param>
-        <param name="max">3.15</param>
-      </command_interface>
+      <command_interface name="position" />
       <state_interface name="position">
         <param name="initial_value">0.0</param>
@@ -587,12 +559,5 @@
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