Commit message: Update robotic arm joint velocities

File: robotic_arm/urdf/robotic_arm.urdf (robot description, URDF)
Before this commit: robot robotic_arm, 9 links, 8 joints
Joints:
- joint eef_joint_l: limit lower=-0.3 upper=0.3 effort=300 velocity=3 -> lower=-0.3 upper=0.3 effort=300 velocity=3.14
- joint eef_joint_r: limit lower=-0.3 upper=0.3 effort=300 velocity=3 -> lower=-0.3 upper=0.3 effort=300 velocity=3.14
- joint joint_1: limit lower=0 upper=6.283 effort=300 velocity=3 -> lower=0 upper=6.283 effort=300 velocity=3.14
- joint joint_2: limit lower=-1.57 upper=1.57 effort=300 velocity=3 -> lower=-1.57 upper=1.57 effort=300 velocity=3.14
- joint joint_3: limit lower=-1.0 upper=4.14 effort=300 velocity=3 -> lower=-1.0 upper=4.14 effort=300 velocity=3.14
- joint joint_4: limit lower=-2.14 upper=2.14 effort=300 velocity=3 -> lower=-2.14 upper=2.14 effort=300 velocity=3.14
- joint joint_5: limit lower=-6.283 upper=6.283 effort=300 velocity=3 -> lower=-6.283 upper=6.283 effort=300 velocity=3.14

Commit message: reset

File: robotic_arm/urdf/robotic_arm.urdf (robot description, URDF)
Before this commit: robot robotic_arm, 9 links, 8 joints
Joints:
- joint eef_joint_l: limit lower=-0.3 upper=0.3 effort=300 velocity=3 -> lower=-0.3 upper=0.3 effort=300 velocity=3.14
- joint eef_joint_r: limit lower=-0.3 upper=0.3 effort=300 velocity=3 -> lower=-0.3 upper=0.3 effort=300 velocity=3.14
- joint joint_1: limit lower=0 upper=6.283 effort=300 velocity=3 -> lower=0 upper=6.283 effort=300 velocity=3.14
- joint joint_2: limit lower=-1.57 upper=1.57 effort=300 velocity=3 -> lower=-1.57 upper=1.57 effort=300 velocity=3.14
- joint joint_3: limit lower=-1.0 upper=4.14 effort=300 velocity=3 -> lower=-1.0 upper=4.14 effort=300 velocity=3.14
- joint joint_4: limit lower=-2.14 upper=2.14 effort=300 velocity=3 -> lower=-2.14 upper=2.14 effort=300 velocity=3.14
- joint joint_5: limit lower=-6.283 upper=6.283 effort=300 velocity=3 -> lower=-6.283 upper=6.283 effort=300 velocity=3.14

File: robotic_arm/urdf/robotic_arm_2.urdf.xacro (robot description, xacro)
@@ -4,5 +4,5 @@
      Commit Version: 1.5.1-0-g916b5db  Build Version: 1.5.7152.31018
      For more information, please see http://wiki.ros.org/sw_urdf_exporter -->
-<robot
+<robot xmlns:xacro="https://wiki.ros.org/xacro.org"
   name="robotic_arm">
   <link name="world" />
@@ -35,19 +35,19 @@
       <geometry>
         <mesh
-          filename="package://robotic_arm/meshes/base_link.STL" />
-      </geometry>
-      <material
-        name="">
-        <color
-          rgba="0.501960784313725 0.501960784313725 0.501960784313725 1" />
-      </material>
-    </visual>
-    <collision>
-      <origin
-        xyz="0 0 0"
-        rpy="0 0 0" />
-      <geometry>
-        <mesh
-          filename="package://robotic_arm/meshes/base_link.STL" />
+          filename="file://$(find robotic_arm)/meshes/base_link.STL" />
+      </geometry>
+      <material
+        name="">
+        <color
+          rgba="0.501960784313725 0.501960784313725 0.501960784313725 1" />
+      </material>
+    </visual>
+    <collision>
+      <origin
+        xyz="0 0 0"
+        rpy="0 0 0" />
+      <geometry>
+        <mesh
+          filename="file://$(find robotic_arm)/meshes/base_link.STL" />
       </geometry>
     </collision>
@@ -76,19 +76,19 @@
       <geometry>
         <mesh
-          filename="package://robotic_arm/meshes/link_1.STL" />
-      </geometry>
-      <material
-        name="">
-        <color
-          rgba="0.501960784313725 0.501960784313725 0.501960784313725 1" />
-      </material>
-    </visual>
-    <collision>
-      <origin
-        xyz="0 0 0"
-        rpy="0 0 0" />
-      <geometry>
-        <mesh
-          filename="package://robotic_arm/meshes/link_1.STL" />
+          filename="file://$(find robotic_arm)/meshes/link_1.STL" />
+      </geometry>
+      <material
+        name="">
+        <color
+          rgba="0.501960784313725 0.501960784313725 0.501960784313725 1" />
+      </material>
+    </visual>
+    <collision>
+      <origin
+        xyz="0 0 0"
+        rpy="0 0 0" />
+      <geometry>
+        <mesh
+          filename="file://$(find robotic_arm)/meshes/link_1.STL" />
       </geometry>
     </collision>
@@ -110,5 +110,5 @@
       upper="6.283"
       effort="300"
-      velocity="3" />
+      velocity="3.14" />
   </joint>
   <link
@@ -135,19 +135,19 @@
       <geometry>
         <mesh
-          filename="package://robotic_arm/meshes/link_2.STL" />
-      </geometry>
-      <material
-        name="">
-        <color
-          rgba="0.501960784313725 0.501960784313725 0.501960784313725 1" />
-      </material>
-    </visual>
-    <collision>
-      <origin
-        xyz="0 0 0"
-        rpy="0 0 0" />
-      <geometry>
-        <mesh
-          filename="package://robotic_arm/meshes/link_2.STL" />
+          filename="file://$(find robotic_arm)/meshes/link_2.STL" />
+      </geometry>
+      <material
+        name="">
+        <color
+          rgba="0.501960784313725 0.501960784313725 0.501960784313725 1" />
+      </material>
+    </visual>
+    <collision>
+      <origin
+        xyz="0 0 0"
+        rpy="0 0 0" />
+      <geometry>
+        <mesh
+          filename="file://$(find robotic_arm)/meshes/link_2.STL" />
       </geometry>
     </collision>
@@ -169,5 +169,5 @@
       upper="1.57"
       effort="300"
-      velocity="3" />
+      velocity="3.14" />
   </joint>
   <link
@@ -194,19 +194,19 @@
       <geometry>
         <mesh
-          filename="package://robotic_arm/meshes/link_3.STL" />
-      </geometry>
-      <material
-        name="">
-        <color
-          rgba="0.501960784313725 0.501960784313725 0.501960784313725 1" />
-      </material>
-    </visual>
-    <collision>
-      <origin
-        xyz="0 0 0"
-        rpy="0 0 0" />
-      <geometry>
-        <mesh
-          filename="package://robotic_arm/meshes/link_3.STL" />
+          filename="file://$(find robotic_arm)/meshes/link_3.STL" />
+      </geometry>
+      <material
+        name="">
+        <color
+          rgba="0.501960784313725 0.501960784313725 0.501960784313725 1" />
+      </material>
+    </visual>
+    <collision>
+      <origin
+        xyz="0 0 0"
+        rpy="0 0 0" />
+      <geometry>
+        <mesh
+          filename="file://$(find robotic_arm)/meshes/link_3.STL" />
       </geometry>
     </collision>
@@ -228,5 +228,5 @@
       upper="4.14"
       effort="300"
-      velocity="3" />
+      velocity="3.14" />
   </joint>
   <link
@@ -253,19 +253,19 @@
       <geometry>
         <mesh
-          filename="package://robotic_arm/meshes/link_4.STL" />
-      </geometry>
-      <material
-        name="">
-        <color
-          rgba="0.501960784313725 0.501960784313725 0.501960784313725 1" />
-      </material>
-    </visual>
-    <collision>
-      <origin
-        xyz="0 0 0"
-        rpy="0 0 0" />
-      <geometry>
-        <mesh
-          filename="package://robotic_arm/meshes/link_4.STL" />
+          filename="file://$(find robotic_arm)/meshes/link_4.STL" />
+      </geometry>
+      <material
+        name="">
+        <color
+          rgba="0.501960784313725 0.501960784313725 0.501960784313725 1" />
+      </material>
+    </visual>
+    <collision>
+      <origin
+        xyz="0 0 0"
+        rpy="0 0 0" />
+      <geometry>
+        <mesh
+          filename="file://$(find robotic_arm)/meshes/link_4.STL" />
       </geometry>
     </collision>
@@ -287,5 +287,5 @@
       upper="2.14"
       effort="300"
-      velocity="3" />
+      velocity="3.14" />
   </joint>
   <link
@@ -312,19 +312,19 @@
       <geometry>
         <mesh
-          filename="package://robotic_arm/meshes/link_5.STL" />
-      </geometry>
-      <material
-        name="">
-        <color
-          rgba="0.501960784313725 0.501960784313725 0.501960784313725 1" />
-      </material>
-    </visual>
-    <collision>
-      <origin
-        xyz="0 0 0"
-        rpy="0 0 0" />
-      <geometry>
-        <mesh
-          filename="package://robotic_arm/meshes/link_5.STL" />
+          filename="file://$(find robotic_arm)/meshes/link_5.STL" />
+      </geometry>
+      <material
+        name="">
+        <color
+          rgba="0.501960784313725 0.501960784313725 0.501960784313725 1" />
+      </material>
+    </visual>
+    <collision>
+      <origin
+        xyz="0 0 0"
+        rpy="0 0 0" />
+      <geometry>
+        <mesh
+          filename="file://$(find robotic_arm)/meshes/link_5.STL" />
       </geometry>
     </collision>
@@ -346,5 +346,5 @@
       upper="6.283"
       effort="300"
-      velocity="3" />
+      velocity="3.14" />
   </joint>
   <link
@@ -371,19 +371,19 @@
       <geometry>
         <mesh
-          filename="package://robotic_arm/meshes/eef_link_r.STL" />
-      </geometry>
-      <material
-        name="">
-        <color
-          rgba="0.501960784313725 0.501960784313725 0.501960784313725 1" />
-      </material>
-    </visual>
-    <collision>
-      <origin
-        xyz="0 0 0"
-        rpy="0 0 0" />
-      <geometry>
-        <mesh
-          filename="package://robotic_arm/meshes/eef_link_r.STL" />
+          filename="file://$(find robotic_arm)/meshes/eef_link_r.STL" />
+      </geometry>
+      <material
+        name="">
+        <color
+          rgba="0.501960784313725 0.501960784313725 0.501960784313725 1" />
+      </material>
+    </visual>
+    <collision>
+      <origin
+        xyz="0 0 0"
+        rpy="0 0 0" />
+      <geometry>
+        <mesh
+          filename="file://$(find robotic_arm)/meshes/eef_link_r.STL" />
       </geometry>
     </collision>
@@ -405,5 +405,5 @@
       upper="0.3"
       effort="300"
-      velocity="3" />
+      velocity="3.14" />
   </joint>
   <link
@@ -430,19 +430,19 @@
       <geometry>
         <mesh
-          filename="package://robotic_arm/meshes/eef_link_l.STL" />
-      </geometry>
-      <material
-        name="">
-        <color
-          rgba="0.501960784313725 0.501960784313725 0.501960784313725 1" />
-      </material>
-    </visual>
-    <collision>
-      <origin
-        xyz="0 0 0"
-        rpy="0 0 0" />
-      <geometry>
-        <mesh
-          filename="package://robotic_arm/meshes/eef_link_l.STL" />
+          filename="file://$(find robotic_arm)/meshes/eef_link_l.STL" />
+      </geometry>
+      <material
+        name="">
+        <color
+          rgba="0.501960784313725 0.501960784313725 0.501960784313725 1" />
+      </material>
+    </visual>
+    <collision>
+      <origin
+        xyz="0 0 0"
+        rpy="0 0 0" />
+      <geometry>
+        <mesh
+          filename="file://$(find robotic_arm)/meshes/eef_link_l.STL" />
       </geometry>
     </collision>
@@ -464,5 +464,5 @@
       upper="0.3"
       effort="300"
-      velocity="3" />
+      velocity="3.14" />
   </joint>
   <transmission name="link_1_trans">
@@ -526,12 +526,63 @@
     </actuator>
   </transmission>
-  <ros2_control name="robotic_arm_controller" type="system">
+  <ros2_control name="GazeboSimSystem" type="system">
+    <hardware>
+      <plugin>mock_components/GenericSystem</plugin>
+    </hardware>
+    <joint name="joint_1">
+      <command_interface name="position" />
+      <state_interface name="position">
+        <param name="initial_value">0.0</param>
+      </state_interface>
+      <state_interface name="velocity" />
+    </joint>
+    <joint name="joint_2">
+      <command_interface name="position" />
+      <state_interface name="position">
+        <param name="initial_value">0.0</param>
+      </state_interface>
+      <state_interface name="velocity" />
+    </joint>
+    <joint name="joint_3">
+      <command_interface name="position" />
+      <state_interface name="position">
+        <param name="initial_value">0.0</param>
+      </state_interface>
+      <state_interface name="velocity" />
+    </joint>
+    <joint name="joint_4">
+      <command_interface name="position" />
+      <state_interface name="position">
+        <param name="initial_value">0.0</param>
+      </state_interface>
+      <state_interface name="velocity" />
+    </joint>
+    <joint name="eef_joint_r">
+      <command_interface name="position" />
+      <state_interface name="position">
+        <param name="initial_value">0.0</param>
+      </state_interface>
+      <state_interface name="velocity" />
+    </joint>
+    <joint name="eef_joint_l">
+      <command_interface name="position"/>
+      <state_interface name="position">
+        <param name="initial_value">0.0</param>
+      </state_interface>
+      <state_interface name="velocity" />
+    </joint>
+    <!-- <joint name="eef_joint_l">
+      <param name="mimic">eef_joint_r</param>
+      <param name="multiplier">-1</param>
+      <command_interface name="position" />
+      <state_interface name="position">
+        <param name="initial_value">0.0</param>
+      </state_interface>
+      <state_interface name="velocity" />
+    </joint> -->
   </ros2_control>
   <gazebo>
     <plugin filename="libgazebo_ros2_control.so" name="gazebo_ros2_control">
-      <robot_param>robot_description</robot_param>
-      <robot_param_node>robot_state_publisher</robot_param_node>
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