Commit message: Reset Again

File: robotic_arm/urdf/robotic_arm copy 2.urdf (robot description, URDF)
Before this commit: robot robotic_arm, 9 links, 8 joints
Links:
- link base_link: geometry collision mesh filename=package://robotic_arm/meshes/base_link.STL; visual mesh filename=package://robotic_arm/meshes/base_link.STL
- link eef_link_l: geometry collision mesh filename=package://robotic_arm/meshes/eef_link_l.STL; visual mesh filename=package://robotic_arm/meshes/eef_link_l.STL
- link eef_link_r: geometry collision mesh filename=package://robotic_arm/meshes/eef_link_r.STL; visual mesh filename=package://robotic_arm/meshes/eef_link_r.STL
- link link_1: geometry collision mesh filename=package://robotic_arm/meshes/link_1.STL; visual mesh filename=package://robotic_arm/meshes/link_1.STL
- link link_2: geometry collision mesh filename=package://robotic_arm/meshes/link_2.STL; visual mesh filename=package://robotic_arm/meshes/link_2.STL
- link link_3: geometry collision mesh filename=package://robotic_arm/meshes/link_3.STL; visual mesh filename=package://robotic_arm/meshes/link_3.STL
- link link_4: geometry collision mesh filename=package://robotic_arm/meshes/link_4.STL; visual mesh filename=package://robotic_arm/meshes/link_4.STL
- link link_5: geometry collision mesh filename=package://robotic_arm/meshes/link_5.STL; visual mesh filename=package://robotic_arm/meshes/link_5.STL
Joints:
- joint eef_joint_l: limit lower=-0.3 upper=0.3 effort=300 velocity=3.14 -> lower=-0.3 upper=0.3 effort=300 velocity=3
- joint eef_joint_r: limit lower=-0.3 upper=0.3 effort=300 velocity=3.14 -> lower=-0.3 upper=0.3 effort=300 velocity=3
- joint joint_1: limit lower=0 upper=6.283 effort=300 velocity=3.14 -> lower=0 upper=6.283 effort=300 velocity=3
- joint joint_2: limit lower=-1.57 upper=1.57 effort=300 velocity=3.14 -> lower=-1.57 upper=1.57 effort=300 velocity=3
- joint joint_3: limit lower=-1.0 upper=4.14 effort=300 velocity=3.14 -> lower=-1.0 upper=4.14 effort=300 velocity=3
- joint joint_4: limit lower=-2.14 upper=2.14 effort=300 velocity=3.14 -> lower=-2.14 upper=2.14 effort=300 velocity=3
- joint joint_5: limit lower=-6.283 upper=6.283 effort=300 velocity=3.14 -> lower=-6.283 upper=6.283 effort=300 velocity=3

File: robotic_arm/urdf/robotic_arm.urdf (robot description, URDF)
Before this commit: robot robotic_arm, 9 links, 8 joints
Joints:
- joint eef_joint_l: limit lower=-0.3 upper=0.3 effort=300 velocity=3.14 -> lower=-0.3 upper=0.3 effort=300 velocity=3
- joint eef_joint_r: limit lower=-0.3 upper=0.3 effort=300 velocity=3.14 -> lower=-0.3 upper=0.3 effort=300 velocity=3
- joint joint_1: limit lower=0 upper=6.283 effort=300 velocity=3.14 -> lower=0 upper=6.283 effort=300 velocity=3
- joint joint_2: limit lower=-1.57 upper=1.57 effort=300 velocity=3.14 -> lower=-1.57 upper=1.57 effort=300 velocity=3
- joint joint_3: limit lower=-1.0 upper=4.14 effort=300 velocity=3.14 -> lower=-1.0 upper=4.14 effort=300 velocity=3
- joint joint_4: limit lower=-2.14 upper=2.14 effort=300 velocity=3.14 -> lower=-2.14 upper=2.14 effort=300 velocity=3
- joint joint_5: limit lower=-6.283 upper=6.283 effort=300 velocity=3.14 -> lower=-6.283 upper=6.283 effort=300 velocity=3
