Commit message: Update robotic_arm configuration and URDF files

File: robotic_arm/urdf/robotic_arm_copy.urdf (robot description, URDF)
Before this commit: robot robotic_arm, 9 links, 8 joints
Links:
- link base_link: geometry collision mesh filename=file://$(find robotic_arm)/meshes/base_link.STL; visual mesh filename=file://$(find robotic_arm)/meshes/base_link.STL
- link eef_link_l: geometry collision mesh filename=file://$(find robotic_arm)/meshes/eef_link_l.STL; visual mesh filename=file://$(find robotic_arm)/meshes/eef_link_l.STL
- link eef_link_r: geometry collision mesh filename=file://$(find robotic_arm)/meshes/eef_link_r.STL; visual mesh filename=file://$(find robotic_arm)/meshes/eef_link_r.STL
- link link_1: geometry collision mesh filename=file://$(find robotic_arm)/meshes/link_1.STL; visual mesh filename=file://$(find robotic_arm)/meshes/link_1.STL
- link link_2: geometry collision mesh filename=file://$(find robotic_arm)/meshes/link_2.STL; visual mesh filename=file://$(find robotic_arm)/meshes/link_2.STL
- link link_3: geometry collision mesh filename=file://$(find robotic_arm)/meshes/link_3.STL; visual mesh filename=file://$(find robotic_arm)/meshes/link_3.STL
- link link_4: geometry collision mesh filename=file://$(find robotic_arm)/meshes/link_4.STL; visual mesh filename=file://$(find robotic_arm)/meshes/link_4.STL
- link link_5: geometry collision mesh filename=file://$(find robotic_arm)/meshes/link_5.STL; visual mesh filename=file://$(find robotic_arm)/meshes/link_5.STL

Commit message: Update kinematics and gripper controllers configuration*** ***Update initial positions for robotic arm*** ***Update material and friction properties of cylinder in arm world

File: robotic_arm/urdf/robotic_arm_copy.urdf (robot description, URDF)
Before this commit: robot robotic_arm, 9 links, 8 joints
Joints:
- joint eef_joint_l: limit lower=-0.5 upper=0.3 effort=300 velocity=3.14 -> lower=-0.5 upper=0.3 effort=0.0 velocity=3.14
- joint eef_joint_r: limit lower=-0.5 upper=0.3 effort=300 velocity=3.14 -> lower=-0.5 upper=0.3 effort=0.0 velocity=3.14
